Commit message: Working on setting up gazebo.

File: description/robot_core.xacro (robot description, xacro)
@@ -47,4 +47,7 @@
     <axis xyz="0 0 1" />
   </joint>
+  <gazebo reference="chassis">
+    <material>Gazebo/White</material>
+  </gazebo>
   <!-- LEFT WHEEL LINK -->
   <link name="left_wheel">
@@ -70,4 +73,7 @@
     <axis xyz="0 0 -1" />
   </joint>
+  <gazebo reference="left_wheel">
+    <material>Gazebo/Blue</material>
+  </gazebo>
   <!-- RIGHT WHEEL LINK -->
   <link name="right_wheel">
@@ -87,4 +93,7 @@
     </xacro:inertial_cylinder>
   </link>
+  <gazebo reference="right_wheel">
+    <material>Gazebo/Blue</material>
+  </gazebo>
   <!-- CASTER WHEEL LINK -->
   <joint name="caster_wheel_joint" type="fixed">
@@ -109,3 +118,6 @@
     </xacro:inertial_sphere>
   </link>
+  <gazebo reference="cahster_wheel">
+    <material>Gazebo/Black</material>
+  </gazebo>
 </robot>
