Commit message: Gazebo working.

File: description/gazebo_control.xacro (robot description, xacro)
@@ -1,22 +1,21 @@
 <?xml version="1.0"?>
 <robot xmlns:xacro="http://www.ros.org/wiki/xacro">
-    <gazebo>
-        <plugin name="diff_drive" filename="libgazebo_ros_diff_drive.so">
-            <!-- Wheel Information -->
-            <left_joint>left_wheel_joint</left_joint>
-            <right_joint>right_wheel_joint
-            </right_joint>
-            <wheel_separation>0.35</wheel_separation>
-            <wheel_diameter>0.1</wheel_diameter>
-            <!-- Limits -->
-            <max_wheel_torque>200</max_wheel_torque>
-            <max_wheel_acceleration>10.0</max_wheel_acceleration>
-            <!-- Output -->
-            <odometry_frame>odom</odometry_frame>
-            <robot_base_frame>base_link</robot_base_frame>
-            <publish_odom>true</publish_odom>
-            <publish_odom_tf>true</publish_odom_tf>
-            <publish_wheel_tf>true</publish_wheel_tf>
-        </plugin>
-    </gazebo>
+  <gazebo>
+    <plugin name="diff_drive" filename="libgazebo_ros_diff_drive.so">
+      <!-- Wheel Information -->
+      <left_joint>left_wheel_joint</left_joint>
+      <right_joint>right_wheel_joint</right_joint>
+      <wheel_separation>0.35</wheel_separation>
+      <wheel_diameter>0.1</wheel_diameter>
+      <!-- Limits -->
+      <max_wheel_torque>200</max_wheel_torque>
+      <max_wheel_acceleration>10.0</max_wheel_acceleration>
+      <!-- Output -->
+      <odometry_frame>odom</odometry_frame>
+      <robot_base_frame>base_link</robot_base_frame>
+      <publish_odom>true</publish_odom>
+      <publish_odom_tf>true</publish_odom_tf>
+      <publish_wheel_tf>true</publish_wheel_tf>
+    </plugin>
+  </gazebo>
 </robot>

File: description/robot_core.xacro (robot description, xacro)
@@ -1,4 +1,4 @@
 <?xml version="1.0"?>
-<robot xmlns:xacro="http://www.ros.org/wiki/xacro" >
+<robot name="my_bot_ddr" xmlns:xacro="http://www.ros.org/wiki/xacro" >
   <xacro:include filename="inertial_macros.xacro"/>
   <material name="white">
@@ -14,4 +14,6 @@
     <color rgba="0 0 0 1" />
   </material>
+  <!-- Over here we include the file that defines extra Gazebo options and motion control driver -->
+  <xacro:include filename="$(find my_bot)/description/robot.xacro.gazebo" />
   <!-- BASE LINK -->
   <link name="base_link">
@@ -41,4 +43,8 @@
     </xacro:inertial_box>
   </link>
+  <!-- <gazebo reference="chassis">
+    <material>Gazebo/White</material>
+  </gazebo> -->
+  <!-- LEFT WHEEL LINK -->
   <joint name="left_wheel_joint" type="continuous">
     <parent link="base_link" />
@@ -47,8 +53,4 @@
     <axis xyz="0 0 1" />
   </joint>
-  <gazebo reference="chassis">
-    <material>Gazebo/White</material>
-  </gazebo>
-  <!-- LEFT WHEEL LINK -->
   <link name="left_wheel">
     <visual>
@@ -56,5 +58,5 @@
         <cylinder radius="0.05" length="0.04" />
       </geometry>
-      <material name="blue"/>
+      <!-- <material name="blue"/> -->
     </visual>
     <collision>
@@ -67,4 +69,8 @@
     </xacro:inertial_cylinder>
   </link>
+  <!-- <gazebo reference="left_wheel">
+    <material>Gazebo/White</material>
+  </gazebo> -->
+  <!-- RIGHT WHEEL LINK -->
   <joint name="right_wheel_joint" type="continuous">
     <parent link="base_link" />
@@ -73,8 +79,4 @@
     <axis xyz="0 0 -1" />
   </joint>
-  <gazebo reference="left_wheel">
-    <material>Gazebo/Blue</material>
-  </gazebo>
-  <!-- RIGHT WHEEL LINK -->
   <link name="right_wheel">
     <visual>
@@ -93,7 +95,7 @@
     </xacro:inertial_cylinder>
   </link>
-  <gazebo reference="right_wheel">
+  <!-- <gazebo reference="right_wheel">
     <material>Gazebo/Blue</material>
-  </gazebo>
+  </gazebo> -->
   <!-- CASTER WHEEL LINK -->
   <joint name="caster_wheel_joint" type="fixed">
@@ -118,6 +120,7 @@
     </xacro:inertial_sphere>
   </link>
-  <gazebo reference="cahster_wheel">
+  <!-- <gazebo reference="cahster_wheel">
     <material>Gazebo/Black</material>
   </gazebo>
+   -->
 </robot>

Commit message: 10-How to get your robot to see in 3D!

File: description/gazebo_control.xacro (robot description, xacro)
@@ -1,23 +1,43 @@
 <?xml version="1.0"?>
-<robot xmlns:xacro="http://www.ros.org/wiki/xacro">
+<robot>
+  <gazebo reference="chassis">
+    <mu1>0.2</mu1>
+    <mu2>0.2</mu2>
+    <material>Gazebo/White</material>
+  </gazebo>
+  <gazebo reference="left_wheel">
+    <mu1>0.2</mu1>
+    <mu2>0.2</mu2>
+    <material>Gazebo/Blue</material>
+  </gazebo>
+  <gazebo reference="right_wheel">
+    <mu1>0.2</mu1>
+    <mu2>0.2</mu2>
+    <material>Gazebo/Blue</material>
+  </gazebo>
+  <gazebo reference="caster_wheel">
+    <mu1>0.000002</mu1>
+    <mu2>0.000002</mu2>
+    <material>Gazebo/Black</material>
+  </gazebo>
   <gazebo>
-    <plugin name="gz::sim::systems::DiffDrive" filename="gz-sim-diff-drive-system">
-      <!-- Wheel Information -->
-      <left_joint>left_wheel_joint</left_joint>
-      <right_joint>right_wheel_joint</right_joint>
-      <wheel_separation>0.297</wheel_separation>
-      <wheel_radius>0.033</wheel_radius>
-      <!-- Limits -->
-      <!-- <max_wheel_torque>200</max_wheel_torque> -->
-      <max_linear_acceleration>0.33</max_linear_acceleration>
-      <!-- Input -->
+    <plugin filename="gz-sim-diff-drive-system" name="gz::sim::systems::DiffDrive">
+      <!-- wheels -->
+      <right_joint>left_wheel_joint</right_joint>
+      <left_joint>right_wheel_joint</left_joint>
+      <!-- kinematics -->
+      <wheel_separation>0.35</wheel_separation>
+      <wheel_diameter>0.1</wheel_diameter>
+      <!-- limits -->
+      <max_linear_acceleration>10</max_linear_acceleration>
+      <!-- topic, frames, and odometry -->
       <topic>cmd_vel</topic>
-      <!-- Output -->
+      <tf_topic>/tf</tf_topic>
+      <odom_topic>odom</odom_topic>
       <frame_id>odom</frame_id>
       <child_frame_id>base_link</child_frame_id>
-      <odom_topic>odom</odom_topic>
       <odom_publisher_frequency>30</odom_publisher_frequency>
-      <tf_topic>/tf</tf_topic>
     </plugin>
+    <!-- Joint state publisher -->
     <plugin filename="gz-sim-joint-state-publisher-system"
       name="gz::sim::systems::JointStatePublisher">

File: description/robot.urdf.xacro (robot description, xacro)
@@ -9,5 +9,8 @@
   <!-- </xacro:unless> -->
   <!-- Over here we include the file that defines extra Gazebo options and motion control driver -->
-  <xacro:include filename="$(find my_bot)/description/robot.xacro.gazebo" />
+  <!-- <xacro:include filename="$(find my_bot)/description/robot.xacro.gazebo" />  -->
+  <xacro:include filename="$(find my_bot)/description/gazebo_control.xacro" />
   <xacro:include filename="$(find my_bot)/description/lidar.xacro" />
+  <!-- <xacro:include filename="$(find my_bot)/description/camera.xacro" /> -->
+  <xacro:include filename="$(find my_bot)/description/depth_camera.xacro" />
 </robot>
