Commit message: Fixed Transformations.

File: description/robot.urdf.xacro (robot description, xacro)
@@ -2,3 +2,5 @@
 <robot xmlns:xacro="http://www.ros.org/wiki/xacro"  name="robot">
   <xacro:include filename="robot_core.xacro" />
+  <!-- Over here we include the file that defines extra Gazebo options and motion control driver -->
+  <!-- <xacro:include filename="$(find my_bot)/description/robot.xacro.gazebo" />   -->
 </robot>

File: description/robot_core.xacro (robot description, xacro)
@@ -1,126 +1,125 @@
 <?xml version="1.0"?>
 <robot name="my_bot_ddr" xmlns:xacro="http://www.ros.org/wiki/xacro" >
-  <xacro:include filename="inertial_macros.xacro"/>
-  <material name="white">
-    <color rgba="1 1 1 1" />
-  </material>
-  <material name="orange">
-    <color rgba="1 0.3 0.1 1" />
-  </material>
-  <material name="blue">
-    <color rgba="0.2 0.2 1 1" />
-  </material>
-  <material name="black">
-    <color rgba="0 0 0 1" />
-  </material>
-  <!-- Over here we include the file that defines extra Gazebo options and motion control driver -->
-  <xacro:include filename="$(find my_bot)/description/robot.xacro.gazebo" />
-  <!-- BASE LINK -->
-  <link name="base_link">
-  </link>
-  <!-- CHASSIS LINK -->
-  <joint name="chassis_joint" type="fixed">
-    <parent link="base_link" />
-    <child link="chassis" />
-    <origin xyz="-0.1 0 0" />
-  </joint>
-  <link name="chassis">
-    <visual>
-      <origin xyz="0.15 0 0.075"/>
-      <geometry>
-        <box size="0.3 0.3 0.15" />
-      </geometry>
-      <material name="white"/>
-    </visual>
-    <collision>
-      <origin xyz="0.15 0 0.075"/>
-      <geometry>
-        <box size="0.3 0.3 0.15" />
-      </geometry>
-    </collision>
-    <xacro:inertial_box mass="0.5" x="0.3" y="0.3" z="0.15">
-      <origin xyz="0.15 0 0.075" rpy="0 0 0"/>
-    </xacro:inertial_box>
-  </link>
-  <!-- <gazebo reference="chassis">
-    <material>Gazebo/White</material>
-  </gazebo> -->
-  <!-- LEFT WHEEL LINK -->
-  <joint name="left_wheel_joint" type="continuous">
-    <parent link="base_link" />
-    <child link="left_wheel" />
-    <origin xyz="0 0.175 0" rpy="-${pi/2} 0 0"/>
-    <axis xyz="0 0 1" />
-  </joint>
-  <link name="left_wheel">
-    <visual>
-      <geometry>
-        <cylinder radius="0.05" length="0.04" />
-      </geometry>
-      <!-- <material name="blue"/> -->
-    </visual>
-    <collision>
-      <geometry>
-        <cylinder radius="0.05" length="0.04" />
-      </geometry>
-    </collision>
-    <xacro:inertial_cylinder mass="0.1" length="0.04" radius="0.01">
-      <origin xyz="0 0 0" rpy="0 0 0"/>
-    </xacro:inertial_cylinder>
-  </link>
-  <!-- <gazebo reference="left_wheel">
-    <material>Gazebo/White</material>
-  </gazebo> -->
-  <!-- RIGHT WHEEL LINK -->
-  <joint name="right_wheel_joint" type="continuous">
-    <parent link="base_link" />
-    <child link="right_wheel" />
-    <origin xyz="0 -0.175 0" rpy="${pi/2} 0 0"/>
-    <axis xyz="0 0 -1" />
-  </joint>
-  <link name="right_wheel">
-    <visual>
-      <geometry>
-        <cylinder radius="0.05" length="0.04" />
-      </geometry>
-      <material name="blue"/>
-    </visual>
-    <collision>
-      <geometry>
-        <cylinder radius="0.05" length="0.04" />
-      </geometry>
-    </collision>
-    <xacro:inertial_cylinder mass="0.1" length="0.04" radius="0.01">
-      <origin xyz="0 0 0" rpy="0 0 0"/>
-    </xacro:inertial_cylinder>
-  </link>
-  <!-- <gazebo reference="right_wheel">
-    <material>Gazebo/Blue</material>
-  </gazebo> -->
-  <!-- CASTER WHEEL LINK -->
-  <joint name="caster_wheel_joint" type="fixed">
-    <parent link="chassis" />
-    <child link="caster_wheel" />
-    <origin xyz="0.24 0 0"/>
-  </joint>
-  <link name="caster_wheel">
-    <visual>
-      <geometry>
-        <sphere radius="0.05"/>
-      </geometry>
-      <material name="black"/>
-    </visual>
-    <collision>
-      <geometry>
-        <sphere radius="0.05"/>
-      </geometry>
-    </collision>
-    <xacro:inertial_sphere mass="0.1" radius="0.05">
-      <origin xyz="0 0 0" rpy="0 0 0"/>
-    </xacro:inertial_sphere>
-  </link>
-  <!-- <gazebo reference="cahster_wheel">
-    <material>Gazebo/Black</material>
-  </gazebo>
-   -->
+    <xacro:include filename="inertial_macros.xacro"/>
+    <xacro:include filename="$(find my_bot)/description/robot.xacro.gazebo" />
+    <material name="white">
+        <color rgba="1 1 1 1" />
+    </material>
+    <material name="orange">
+        <color rgba="1 0.3 0.1 1"/>
+    </material>
+    <material name="blue">
+        <color rgba="0.2 0.2 1 1"/>
+    </material>
+    <material name="black">
+        <color rgba="0 0 0 1"/>
+    </material>
+    <!-- BASE LINK -->
+    <link name="base_link"></link>
+    <!-- CHASSIS LINK -->
+    <joint name="chassis_joint" type="fixed">
+        <parent link="base_link"/>
+        <child link="chassis"/>
+        <origin xyz="-0.1 0 0"/>
+    </joint>
+    <link name="chassis">
+        <visual>
+            <origin xyz="0.15 0 0.075"/>
+            <geometry>
+                <box size="0.3 0.3 0.15"/>
+            </geometry>
+            <material name="white"/>
+        </visual>
+        <collision>
+            <origin xyz="0.15 0 0.075"/>
+            <geometry>
+                <box size="0.3 0.3 0.15"/>
+            </geometry>
+        </collision>
+        <xacro:inertial_box mass="0.5" x="0.3" y="0.3" z="0.15">
+            <origin xyz="0.15 0 0.075" rpy="0 0 0"/>
+        </xacro:inertial_box>
+    </link>
+    <!-- <gazebo reference="chassis">
+        <material>Gazebo/White</material>
+    </gazebo> -->
+    <!-- LEFT WHEEL LINK -->
+    <joint name="left_wheel_joint" type="continuous">
+        <parent link="chassis"/>
+        <child link="left_wheel"/>
+        <origin xyz="0 0.175 0" rpy="-${pi/2} 0 0" />
+        <axis xyz="0 0 1"/>
+    </joint>
+    <link name="left_wheel">
+        <visual>
+            <geometry>
+                <cylinder radius="0.05" length="0.04"/>
+            </geometry>
+            <material name="blue"/>
+        </visual>
+        <collision>
+            <geometry>
+                <cylinder radius="0.05" length="0.04"/>
+            </geometry>
+        </collision>
+        <xacro:inertial_cylinder mass="0.1" length="0.04" radius="0.05">
+            <origin xyz="0 0 0" rpy="0 0 0"/>
+        </xacro:inertial_cylinder>
+    </link>
+    <!-- <gazebo reference="left_wheel">
+        <material>Gazebo/Blue</material>
+    </gazebo> -->
+    <!-- RIGHT WHEEL LINK -->
+    <joint name="right_wheel_joint" type="continuous">
+        <parent link="chassis"/>
+        <child link="right_wheel"/>
+        <origin xyz="0 -0.175 0" rpy="${pi/2} 0 0" />
+        <axis xyz="0 0 -1"/>
+    </joint>
+    <link name="right_wheel">
+        <visual>
+            <geometry>
+                <cylinder radius="0.05" length="0.04"/>
+            </geometry>
+            <material name="blue"/>
+        </visual>
+        <collision>
+            <geometry>
+                <cylinder radius="0.05" length="0.04"/>
+            </geometry>
+        </collision>
+        <xacro:inertial_cylinder mass="0.1" length="0.04" radius="0.05">
+            <origin xyz="0 0 0" rpy="0 0 0"/>
+        </xacro:inertial_cylinder>
+    </link>
+    <!-- <gazebo reference="right_wheel">
+        <material>Gazebo/Blue</material>
+    </gazebo> -->
+    <!-- CASTER WHEEL LINK -->
+    <joint name="caster_wheel_joint" type="fixed">
+        <parent link="chassis"/>
+        <child link="caster_wheel"/>
+        <origin xyz="0.24 0 0"/>
+    </joint>
+    <link name="caster_wheel">
+        <visual>
+            <geometry>
+                <sphere radius="0.05"/>
+            </geometry>
+            <material name="black"/>
+        </visual>
+        <collision>
+            <geometry>
+                <sphere radius="0.05"/>
+            </geometry>
+        </collision>
+        <xacro:inertial_sphere mass="0.1" radius="0.05">
+            <origin xyz="0 0 0" rpy="0 0 0"/>
+        </xacro:inertial_sphere>
+    </link>
+    <!-- <gazebo reference="caster_wheel">
+        <material>Gazebo/Black</material>
+        <mu1 value="0.001"/>
+        <mu2 value="0.001"/>
+    </gazebo> -->
 </robot>

Commit message: Completed How do we add LIDAR to a ROS robot?

File: description/robot.urdf.xacro (robot description, xacro)
@@ -2,5 +2,12 @@
 <robot xmlns:xacro="http://www.ros.org/wiki/xacro"  name="robot">
   <xacro:include filename="robot_core.xacro" />
+  <!-- <xacro:if value="$(arg use_ros2_control)">
+    <xacro:include filename="ros2_control.xacro" />
+  </xacro:if> -->
+  <!-- <xacro:unless value="$(arg use_ros2_control)"> -->
+    <!-- <xacro:include filename="gazebo_control.xacro" /> -->
+  <!-- </xacro:unless> -->
   <!-- Over here we include the file that defines extra Gazebo options and motion control driver -->
   <xacro:include filename="$(find my_bot)/description/robot.xacro.gazebo" />
+  <xacro:include filename="$(find my_bot)/description/lidar.xacro" />
 </robot>

File: description/robot_core.xacro (robot description, xacro)
@@ -13,4 +13,7 @@
   <material name="black">
     <color rgba="0 0 0 1"/>
+  </material>
+  <material name="red">
+    <color rgba="1 0 0 1"/>
   </material>
   <!-- BASE LINK -->

Commit message: Working on Nav2.

File: description/robot.urdf.xacro (robot description, xacro)
@@ -9,6 +9,6 @@
   <!-- </xacro:unless> -->
   <!-- Over here we include the file that defines extra Gazebo options and motion control driver -->
-  <!-- <xacro:include filename="$(find my_bot)/description/gazebo_control.xacro" />  -->
-  <xacro:include filename="$(find my_bot)/description/ros2_control.xacro" />
+  <xacro:include filename="$(find my_bot)/description/gazebo_control.xacro" />
+  <!-- <xacro:include filename="$(find my_bot)/description/ros2_control.xacro" />  -->
   <xacro:include filename="$(find my_bot)/description/lidar.xacro" />
   <xacro:include filename="$(find my_bot)/description/camera.xacro" />

File: description/robot_core.xacro (robot description, xacro)
@@ -19,4 +19,12 @@
   <!-- BASE LINK -->
   <link name="base_link"></link>
+  <!-- BASE_FOOTPRINT LINK -->
+  <joint name="base_footprint_joint" type="fixed">
+    <parent link="base_link"/>
+    <child link="base_footprint"/>
+    <origin xyz="0 0 0" rpy="0 0 0"/>
+  </joint>
+  <link name="base_footprint">
+  </link>
   <!-- CHASSIS LINK -->
   <joint name="chassis_joint" type="fixed">
@@ -59,5 +67,6 @@
     <collision>
       <geometry>
-        <cylinder radius="0.05" length="0.04"/>
+        <!-- <cylinder radius="0.05" length="0.04"/> -->
+        <sphere radius="0.05" />
       </geometry>
     </collision>
@@ -82,5 +91,6 @@
     <collision>
       <geometry>
-        <cylinder radius="0.05" length="0.04"/>
+        <!-- <cylinder radius="0.05" length="0.04"/> -->
+        <sphere radius="0.05" />
       </geometry>
     </collision>
